Commit message: removed unnecessary configurations

File: Simulation/urdf/arlo_2stack.urdf.xacro (robot description, xacro)
@@ -353,5 +353,5 @@
     <joint name="camera_joint" type="fixed">
 	  <axis xyz="0 1 0" />
-	  <origin xyz="0.18 0 0.45" rpy="0 0.785398163 0"/>
+	  <origin xyz="0.18 0 0.45" rpy="0 0.785398 0"/>
 	  <parent link="base_link"/>
 	  <child link="camera_link"/>
@@ -370,5 +370,4 @@
 			<box size="${camera_link} ${camera_link} ${camera_link}"/>
 	    </geometry>
-	    <material name="red"/>
 	  </visual>
 	  <inertial>

Commit message: small fixes and cleanup

File: Simulation/urdf/arlo_2stack.urdf.xacro (robot description, xacro)
@@ -1,3 +1,6 @@
 <?xml version="1.0"?>
+<!-- modified by Tristan Schwörer -->
+<!-- added gazebo plugins for Lidar, Camera and diffwheel drive -->
+<!-- removed not needed joints and links of nonexistend hardware -->
 <robot name="arlobot_hardware" xmlns:xacro="http://ros.org/wiki/xacro">
   <!-- Macro for ArloBot body. -->
@@ -265,65 +268,4 @@
       <joint_properties damping="0.0" friction="0.0"/>
     </joint>
-    <!-- This pretends to be in the center in order to aid in calculating degrees from multiple sensors on one fake laser scan -->
-    <joint name="ping_array_joint" type="fixed">
-      <origin xyz="0 0 0.03695" rpy="0 0 0"/>
-      <parent link="base_link"/>
-      <child link="ping_sensor_array"/>
-    </joint>
-    <link name="ping_sensor_array">
-      <visual>
-        <geometry>
-          <box size="0.0174 0.06 0.0644"/>
-        </geometry>
-      </visual>
-      <inertial>
-        <mass value="0.001"/>
-        <origin xyz="0 0 0"/>
-        <inertia ixx="0.0001" ixy="0.0" ixz="0.0"
-                 iyy="0.0001" iyz="0.0"
-                 izz="0.0001"/>
-      </inertial>
-    </link>
-    <joint name="ir_array_joint" type="fixed">
-      <origin xyz="0 0 0.03695" rpy="0 0 0"/>
-      <parent link="base_link"/>
-      <child link="ir_sensor_array"/>
-    </joint>
-    <link name="ir_sensor_array">
-      <visual>
-        <geometry>
-          <box size="0.0174 0.06 0.0644"/>
-        </geometry>
-      </visual>
-      <inertial>
-        <mass value="0.001"/>
-        <origin xyz="0 0 0"/>
-        <inertia ixx="0.0001" ixy="0.0" ixz="0.0"
-                 iyy="0.0001" iyz="0.0"
-                 izz="0.0001"/>
-      </inertial>
-    </link>
-    <!-- Scanse Sweep Sensor on top of robot -->
-    <joint name="scanse_sweep_joint" type="fixed">
-      <!-- Minor adjustments based on lining up Scanse Sweep output with 3D Sensor output -->
-      <!-- So if the 3D sensor is misaligned the Scanse Sweep is off by the same amount -->
-      <origin xyz="0.15 0.0 0.269107" rpy="0 0 3.13"/>
-      <parent link="base_link"/>
-      <child link="scanse_sweep"/>
-    </joint>
-    <link name="scanse_sweep">
-      <visual>
-        <geometry>
-          <box size="0.0 0.0 0.0"/>
-        </geometry>
-      </visual>
-      <inertial>
-        <mass value="0.001"/>
-        <origin xyz="0 0 0"/>
-        <inertia ixx="0.0001" ixy="0.0" ixz="0.0"
-                 iyy="0.0001" iyz="0.0"
-                 izz="0.0001"/>
-      </inertial>
-    </link>
 	<link name="hokuyo_link">
       <collision>
@@ -353,5 +295,5 @@
     <joint name="camera_joint" type="fixed">
 	  <axis xyz="0 1 0" />
-	  <origin xyz="0.18 0 0.45" rpy="0 0.785398 0"/>
+	  <origin xyz="0.18 0 0.45" rpy="0 0.733038 0"/>
 	  <parent link="base_link"/>
 	  <child link="camera_link"/>
@@ -377,32 +319,4 @@
 	  </inertial>
 	</link>
-    <!-- RPLIDAR on top of robot -->
-    <joint name="rplidar_joint" type="fixed">
-      <!-- WARNING: The 'rpy' means Roll, Pitch, Yaw, but in the static_transform_publisher the order -->
-      <!-- is Yaw, Pitch, Roll !!!  So don't forget to translate those! -->
-      <!-- The best way to tweak this is to delete this section, start the robot, and use -->
-      <!-- staticTransformExample.sh to broadcast this transform while watching in RVIZ, -->
-      <!-- and keep tweaking the numbers and killing and restarting that transform broadcaster. -->
-      <!-- NOTE: The "FRONT" of the RPLIDAR A2/3 is the point where the cord comes out. -->
-      <!-- Hence the r of 3.1 to rotate it half way around.  -->
-      <!-- The height is set even with the top plate. It shouldn't matter really. -->
-      <origin xyz="0.125 0.0 0.269107" rpy="0.0 0.0 0.0"/>
-      <parent link="base_link"/>
-      <child link="rplidar"/>
-    </joint>
-    <link name="rplidar">
-      <visual>
-        <geometry>
-          <box size="0.0 0.0 0.0"/>
-        </geometry>
-      </visual>
-      <inertial>
-        <mass value="0.001"/>
-        <origin xyz="0 0 0"/>
-        <inertia ixx="0.0001" ixy="0.0" ixz="0.0"
-                 iyy="0.0001" iyz="0.0"
-                 izz="0.0001"/>
-      </inertial>
-    </link>
   </xacro:macro>
   <xacro:macro name="arlobot_standoff_5in" params="parent number x_loc y_loc z_loc">

Commit message: Fixed caster size added turning joint for caster wheel

File: Simulation/urdf/arlo_2stack.urdf.xacro (robot description, xacro)
@@ -93,5 +93,5 @@
       </inertial>
       <visual>
-        <origin xyz="0 0 0" rpy="-1.5707 0 1.5707"/>
+        <origin xyz="0 0.02 0.050625" rpy="-1.5707 0 0"/>
         <geometry>
           <mesh filename="package://arlobot_ros/meshes/28971-Caster-Wheel-Kit-v1.0_simplified.stl"/>
@@ -102,7 +102,7 @@
       </visual>
       <collision>
-        <origin xyz="0 0 0" rpy="-1.5707 0 1.5707"/>
-        <geometry>
-          <mesh filename="package://arlobot_ros/meshes/28971-Caster-Wheel-Kit-v1.0_simplified.stl"/>
+        <origin xyz="0 0.02 0" rpy="-1.5707 0 1.5707"/>
+        <geometry>
+    	  <sphere radius="0.050625"/>
         </geometry>
         <material name="light_grey">
@@ -111,6 +111,7 @@
       </collision>
     </link>
-    <joint name="front_caster_joint" type="fixed">
-      <origin xyz="0.18745 0 -0.002875" rpy="0 0 0"/>
+    <joint name="front_caster_joint" type="continuous">
+      <axis xyz="0 0 1" rpy="0 0 0" />
+      <origin xyz="0.18745 -0.02 -0.050625" rpy="0 0 0"/>
       <parent link="base_link"/>
       <child link="front_caster"/>
@@ -125,5 +126,5 @@
       </inertial>
       <visual>
-        <origin xyz="0 0 0" rpy="-1.5707 0 1.5707"/>
+        <origin xyz="0 0.02 0.050625" rpy="-1.5707 0 0"/>
         <geometry>
           <mesh filename="package://arlobot_ros/meshes/28971-Caster-Wheel-Kit-v1.0_simplified.stl"/>
@@ -134,7 +135,7 @@
       </visual>
       <collision>
-        <origin xyz="0 0 0" rpy="-1.5707 0 1.5707"/>
-        <geometry>
-          <mesh filename="package://arlobot_ros/meshes/28971-Caster-Wheel-Kit-v1.0_simplified.stl"/>
+        <origin xyz="0 0.02 0" rpy="-1.5707 0 1.5707"/>
+        <geometry>
+    	  <sphere radius="0.050625"/>
         </geometry>
         <material name="light_grey">
@@ -143,7 +144,7 @@
       </collision>
     </link>
-	<!-- modified by Tristan Schwoerer -->
-    <joint name="rear_caster_joint" type="fixed">
-      <origin xyz="-0.18745 0 -0.002875" rpy="0 0 0"/>
+    <joint name="rear_caster_joint" type="continuous">
+      <axis xyz="0 0 1" rpy="0 0 0" />
+      <origin xyz="-0.18745 -0.02 -0.050625" rpy="0 0 0"/>
       <parent link="base_link"/>
       <child link="rear_caster"/>
@@ -227,4 +228,12 @@
           <cylinder radius="0.0762" length="0.03175"/>
         </geometry>
+        <surface>
+	        <friction>
+	          <ode>
+	            <mu>100.00</mu>
+	            <mu2>50.00</mu2>
+	          </ode>
+	        </friction>
+        </surface>
       </collision>
     </link>
@@ -257,4 +266,12 @@
           <cylinder radius="0.0762" length="0.03175"/>
         </geometry>
+        <surface>
+	        <friction>
+	          <ode>
+	            <mu>100.00</mu>
+	            <mu2>50.00</mu2>
+	          </ode>
+	        </friction>
+        </surface>
       </collision>
     </link>
@@ -295,5 +312,5 @@
     <joint name="camera_joint" type="fixed">
 	  <axis xyz="0 1 0" />
-	  <origin xyz="0.18 0 0.45" rpy="0 0.733038 0"/>
+	  <origin xyz="0.18 0 0.45" rpy="0 0.785398 0"/>
 	  <parent link="base_link"/>
 	  <child link="camera_link"/>

Commit message: removed 3rd layer

File: Simulation/urdf/arlo_2stack.urdf.xacro (robot description, xacro)
@@ -312,5 +312,5 @@
     <joint name="camera_joint" type="fixed">
 	  <axis xyz="0 1 0" />
-	  <origin xyz="0.18 0 0.45" rpy="0 0.785398 0"/>
+	  <origin xyz="0.18 0 0.34875" rpy="0 0.785398 0"/>
 	  <parent link="base_link"/>
 	  <child link="camera_link"/>
@@ -406,41 +406,4 @@
     <xacro:arlobot_standoff_5in parent="${parent}" number="3" x_loc="-0.052832" y_loc="0.1314196"
                           z_loc="0.06825"/>
-    <joint name="plate_1_joint" type="fixed">
-      <origin xyz="0 0 0.1365" rpy="0 0 0"/>
-      <parent link="plate_0_link"/>
-      <child link="plate_1_link"/>
-    </joint>
-    <link name="plate_1_link">
-      <inertial>
-        <mass value="0.01"/>
-        <origin xyz="0 0 0"/>
-        <inertia ixx="0.01" ixy="0.0" ixz="0.0"
-                 iyy="0.01" iyz="0.0"
-                 izz="0.01"/>
-      </inertial>
-      <visual>
-        <origin xyz=" 0 0 0 " rpy="0 0 0"/>
-        <geometry>
-          <cylinder length="0.0095" radius="0.2245"/>
-        </geometry>
-        <material name="veryDarkGrey">
-          <color rgba=".2 .2 .2 1"/>
-        </material>
-      </visual>
-      <collision>
-        <origin xyz="0.0 0.0 0.0" rpy="0 0 0"/>
-        <geometry>
-          <cylinder length="0.0095" radius="0.2245"/>
-        </geometry>
-      </collision>
-    </link>
-    <xacro:arlobot_standoff_5in parent="plate_0_link" number="4" x_loc="0.0676402" y_loc="0.1314196"
-                          z_loc="0.06825"/>
-    <xacro:arlobot_standoff_5in parent="plate_0_link" number="5" x_loc="0.0676402" y_loc="-0.1314196"
-                          z_loc="0.06825"/>
-    <xacro:arlobot_standoff_5in parent="plate_0_link" number="6" x_loc="-0.052832" y_loc="-0.1314196"
-                          z_loc="0.06825"/>
-    <xacro:arlobot_standoff_5in parent="plate_0_link" number="7" x_loc="-0.052832" y_loc="0.1314196"
-                          z_loc="0.06825"/>
   </xacro:macro>
 </robot>

Commit message: included stl file in own meshes folder fixed core count to be compatible with most systems

File: Simulation/urdf/arlo_2stack.urdf.xacro (robot description, xacro)
@@ -95,5 +95,5 @@
         <origin xyz="0 0.02 0.050625" rpy="-1.5707 0 0"/>
         <geometry>
-          <mesh filename="package://arlobot_ros/meshes/28971-Caster-Wheel-Kit-v1.0_simplified.stl"/>
+          <mesh filename="package://Simulation/meshes/28971-Caster-Wheel-Kit-v1.0_simplified.stl"/>
         </geometry>
         <material name="light_grey">
@@ -128,5 +128,5 @@
         <origin xyz="0 0.02 0.050625" rpy="-1.5707 0 0"/>
         <geometry>
-          <mesh filename="package://arlobot_ros/meshes/28971-Caster-Wheel-Kit-v1.0_simplified.stl"/>
+          <mesh filename="package://Simulation/meshes/28971-Caster-Wheel-Kit-v1.0_simplified.stl"/>
         </geometry>
         <material name="light_grey">

Commit message: Included IMU fixed diff drive

File: Simulation/urdf/arlo_2stack.urdf.xacro (robot description, xacro)
@@ -309,4 +309,29 @@
       <parent link="base_link"/>
       <child link="hokuyo_link"/>
+    </joint>
+	<link name="imu_link">
+      <collision>
+        <origin xyz="0 0 0" rpy="0 0 0"/>
+        <geometry>
+          <box size="0.1 0.1 0.1"/>
+        </geometry>
+      </collision>
+      <visual>
+        <origin xyz="0 0 0" rpy="0 0 0"/>
+        <geometry>
+          <box size="0.05 0.05 0.05"/>
+        </geometry>
+      </visual>
+      <inertial>
+        <mass value="1e-5" />
+        <origin xyz="0 0 0" rpy="0 0 0"/>
+        <inertia ixx="1e-6" ixy="0" ixz="0" iyy="1e-6" iyz="0" izz="1e-6" />
+      </inertial>
+    </link>
+    <joint name="imu_joint" type="fixed">
+      <!--<axis xyz="0 0 0" />-->
+      <origin xyz="0 0 0" rpy="0 0 0"/>
+      <parent link="base_link"/>
+      <child link="imu_link"/>
     </joint>
     <joint name="camera_joint" type="fixed">

Commit message: cleanup in robot description and removed small failures

File: Simulation/urdf/arlo_2stack.urdf.xacro (robot description, xacro)
@@ -93,5 +93,5 @@
       </inertial>
       <visual>
-        <origin xyz="0 0.02 0.050625" rpy="-1.5707 0 0"/>
+        <origin xyz="0 0.02 0.050625" rpy="-1.570796327 0 0"/>
         <geometry>
           <mesh filename="package://Simulation/meshes/28971-Caster-Wheel-Kit-v1.0_simplified.stl"/>
@@ -102,5 +102,5 @@
       </visual>
       <collision>
-        <origin xyz="0 0.02 0" rpy="-1.5707 0 1.5707"/>
+        <origin xyz="0 0.02 0" rpy="-1.570796327 0 1.570796327"/>
         <geometry>
     	  <sphere radius="0.050625"/>
@@ -126,5 +126,5 @@
       </inertial>
       <visual>
-        <origin xyz="0 0.02 0.050625" rpy="-1.5707 0 0"/>
+        <origin xyz="0 0.02 0.050625" rpy="-1.570796327 0 0"/>
         <geometry>
           <mesh filename="package://Simulation/meshes/28971-Caster-Wheel-Kit-v1.0_simplified.stl"/>
@@ -135,5 +135,5 @@
       </visual>
       <collision>
-        <origin xyz="0 0.02 0" rpy="-1.5707 0 1.5707"/>
+        <origin xyz="0 0.02 0" rpy="-1.570796327 0 1.570796327"/>
         <geometry>
     	  <sphere radius="0.050625"/>
@@ -163,5 +163,5 @@
       </inertial>
       <visual>
-        <origin xyz="0 0 0" rpy="0 1.5707 1.5707"/>
+        <origin xyz="0 0 0" rpy="0 1.570796327 1.570796327"/>
         <geometry>
           <cylinder radius="0.00635" length="0.00635"/>
@@ -170,5 +170,5 @@
       </visual>
       <collision>
-        <origin xyz="0 0 0" rpy="0 1.5707 1.5707"/>
+        <origin xyz="0 0 0" rpy="0 1.570796327 1.570796327"/>
         <geometry>
           <cylinder radius="0.00635" length="0.00635"/>
@@ -190,5 +190,5 @@
       </inertial>
       <visual>
-        <origin xyz="0 0 0" rpy="0 1.5707 1.5707"/>
+        <origin xyz="0 0 0" rpy="0 1.570796327 1.570796327"/>
         <geometry>
           <cylinder radius="0.00635" length="0.00635"/>
@@ -197,5 +197,5 @@
       </visual>
       <collision>
-        <origin xyz="0 0 0" rpy="0 1.5707 1.5707"/>
+        <origin xyz="0 0 0" rpy="0 1.570796327 1.570796327"/>
         <geometry>
           <cylinder radius="0.00635" length="0.00635"/>
@@ -217,5 +217,5 @@
       </inertial>
       <visual>
-        <origin xyz="0 0 0" rpy="0 1.5707 1.5707"/>
+        <origin xyz="0 0 0" rpy="0 1.570796327 1.570796327"/>
         <geometry>
           <cylinder radius="0.0762" length="0.03175"/>
@@ -224,5 +224,5 @@
       </visual>
       <collision>
-        <origin xyz="0 0 0" rpy="0 1.5707 1.5707"/>
+        <origin xyz="0 0 0" rpy="0 1.570796327 1.570796327"/>
         <geometry>
           <cylinder radius="0.0762" length="0.03175"/>
@@ -255,5 +255,5 @@
       </inertial>
       <visual>
-        <origin xyz="0 0 0" rpy="0 1.5707 1.5707"/>
+        <origin xyz="0 0 0" rpy="0 1.570796327 1.570796327"/>
         <geometry>
           <cylinder radius="0.0762" length="0.03175"/>
@@ -262,5 +262,5 @@
       </visual>
       <collision>
-        <origin xyz="0 0 0" rpy="0 1.5707 1.5707"/>
+        <origin xyz="0 0 0" rpy="0 1.570796327 1.570796327"/>
         <geometry>
           <cylinder radius="0.0762" length="0.03175"/>
