Commit message: URDF cleanup
moved links and joints of sensors to separate macros
separate sensor macros are now fully parameter controllable

File: Simulation/urdf/arlo_stack.urdf.xacro (robot description, xacro)
@@ -1,6 +1,3 @@
 <?xml version="1.0"?>
-<!-- modified by Tristan Schwörer -->
-<!-- added gazebo plugins for Lidar, Camera and diffwheel drive -->
-<!-- removed not needed joints and links of nonexistend hardware -->
 <robot name="arlobot_hardware" xmlns:xacro="http://ros.org/wiki/xacro">
   <!-- Macro for ArloBot body. -->
@@ -93,5 +90,5 @@
       </inertial>
       <visual>
-        <origin xyz="0 0.02 0.050625" rpy="-1.570796327 0 0"/>
+        <origin xyz="0 0.02 0.050625" rpy="${-M_PI/2} 0 ${M_PI/2}"/>
         <geometry>
           <mesh filename="package://Simulation/meshes/28971-Caster-Wheel-Kit-v1.0_simplified.stl"/>
@@ -102,5 +99,5 @@
       </visual>
       <collision>
-        <origin xyz="0 0.02 0" rpy="-1.570796327 0 1.570796327"/>
+        <origin xyz="0 0.02 0" rpy="${-M_PI/2} 0 ${M_PI/2}"/>
         <geometry>
     	  <sphere radius="0.050625"/>
@@ -126,5 +123,5 @@
       </inertial>
       <visual>
-        <origin xyz="0 0.02 0.050625" rpy="-1.570796327 0 0"/>
+        <origin xyz="0 0.02 0.050625" rpy="${-M_PI/2} 0 ${M_PI/2}"/>
         <geometry>
           <mesh filename="package://Simulation/meshes/28971-Caster-Wheel-Kit-v1.0_simplified.stl"/>
@@ -135,5 +132,5 @@
       </visual>
       <collision>
-        <origin xyz="0 0.02 0" rpy="-1.570796327 0 1.570796327"/>
+        <origin xyz="0 0.02 0" rpy="${-M_PI/2} 0 ${M_PI/2}"/>
         <geometry>
     	  <sphere radius="0.050625"/>
@@ -163,5 +160,5 @@
       </inertial>
       <visual>
-        <origin xyz="0 0 0" rpy="0 1.570796327 1.570796327"/>
+        <origin xyz="0 0 0" rpy="0 ${M_PI/2} ${M_PI/2}"/>
         <geometry>
           <cylinder radius="0.00635" length="0.00635"/>
@@ -170,5 +167,5 @@
       </visual>
       <collision>
-        <origin xyz="0 0 0" rpy="0 1.570796327 1.570796327"/>
+        <origin xyz="0 0 0" rpy="0 ${M_PI/2} ${M_PI/2}"/>
         <geometry>
           <cylinder radius="0.00635" length="0.00635"/>
@@ -190,5 +187,5 @@
       </inertial>
       <visual>
-        <origin xyz="0 0 0" rpy="0 1.570796327 1.570796327"/>
+        <origin xyz="0 0 0" rpy="0 ${M_PI/2} ${M_PI/2}"/>
         <geometry>
           <cylinder radius="0.00635" length="0.00635"/>
@@ -197,5 +194,5 @@
       </visual>
       <collision>
-        <origin xyz="0 0 0" rpy="0 1.570796327 1.570796327"/>
+        <origin xyz="0 0 0" rpy="0 ${M_PI/2} ${M_PI/2}"/>
         <geometry>
           <cylinder radius="0.00635" length="0.00635"/>
@@ -217,5 +214,5 @@
       </inertial>
       <visual>
-        <origin xyz="0 0 0" rpy="0 1.570796327 1.570796327"/>
+        <origin xyz="0 0 0" rpy="0 ${M_PI/2} ${M_PI/2}"/>
         <geometry>
           <cylinder radius="0.0762" length="0.03175"/>
@@ -224,5 +221,5 @@
       </visual>
       <collision>
-        <origin xyz="0 0 0" rpy="0 1.570796327 1.570796327"/>
+        <origin xyz="0 0 0" rpy="0 ${M_PI/2} ${M_PI/2}"/>
         <geometry>
           <cylinder radius="0.0762" length="0.03175"/>
@@ -255,5 +252,5 @@
       </inertial>
       <visual>
-        <origin xyz="0 0 0" rpy="0 1.570796327 1.570796327"/>
+        <origin xyz="0 0 0" rpy="0 ${M_PI/2} ${M_PI/2}"/>
         <geometry>
           <cylinder radius="0.0762" length="0.03175"/>
@@ -262,5 +259,5 @@
       </visual>
       <collision>
-        <origin xyz="0 0 0" rpy="0 1.570796327 1.570796327"/>
+        <origin xyz="0 0 0" rpy="0 ${M_PI/2} ${M_PI/2}"/>
         <geometry>
           <cylinder radius="0.0762" length="0.03175"/>
@@ -285,80 +282,4 @@
       <joint_properties damping="0.0" friction="0.0"/>
     </joint>
-	<link name="hokuyo_link">
-      <collision>
-        <origin xyz="0 0 0" rpy="0 0 0"/>
-        <geometry>
-          <box size="0.1 0.1 0.1"/>
-        </geometry>
-      </collision>
-      <visual>
-        <origin xyz="0 0 0" rpy="0 0 0"/>
-        <geometry>
-          <mesh filename="package://Simulation/meshes/hokuyo.dae"/>
-        </geometry>
-      </visual>
-      <inertial>
-        <mass value="1e-5" />
-        <origin xyz="0 0 0" rpy="0 0 0"/>
-        <inertia ixx="1e-6" ixy="0" ixz="0" iyy="1e-6" iyz="0" izz="1e-6" />
-      </inertial>
-    </link>
-    <joint name="hokuyo_joint" type="fixed">
-      <!--<axis xyz="0 0 1" />-->
-      <origin xyz="0.175 0 0.035" rpy="0 0 0"/>
-      <parent link="base_link"/>
-      <child link="hokuyo_link"/>
-    </joint>
-	<link name="imu_link">
-      <collision>
-        <origin xyz="0 0 0" rpy="0 0 0"/>
-        <geometry>
-          <box size="0.1 0.1 0.1"/>
-        </geometry>
-      </collision>
-      <visual>
-        <origin xyz="0 0 0" rpy="0 0 0"/>
-        <geometry>
-          <box size="0.05 0.05 0.05"/>
-        </geometry>
-      </visual>
-      <inertial>
-        <mass value="1e-5" />
-        <origin xyz="0 0 0" rpy="0 0 0"/>
-        <inertia ixx="1e-6" ixy="0" ixz="0" iyy="1e-6" iyz="0" izz="1e-6" />
-      </inertial>
-    </link>
-    <joint name="imu_joint" type="fixed">
-      <!--<axis xyz="0 0 0" />-->
-      <origin xyz="0 0 0" rpy="0 0 0"/>
-      <parent link="base_link"/>
-      <child link="imu_link"/>
-    </joint>
-    <joint name="camera_joint" type="fixed">
-	  <axis xyz="0 1 0" />
-	  <origin xyz="0.18 0 0.34875" rpy="0 0.785398 0"/>
-	  <parent link="base_link"/>
-	  <child link="camera_link"/>
-	</joint>
-	<!-- Camera -->
-	<link name="camera_link">
-	  <collision>
-	    <origin xyz="0 0 0" rpy="0 0 0"/>
-	    <geometry>
-			<box size="${camera_link} ${camera_link} ${camera_link}"/>
-	  	</geometry>
-	  </collision>
-	  <visual>
-	    <origin xyz="0 0 0" rpy="0 0 0"/>
-	    <geometry>
-			<box size="${camera_link} ${camera_link} ${camera_link}"/>
-	    </geometry>
-	  </visual>
-	  <inertial>
-	    <mass value="1e-5" />
-	    <origin xyz="0 0 0" rpy="0 0 0"/>
-	    <inertia ixx="1e-6" ixy="0" ixz="0" iyy="1e-6" iyz="0" izz="1e-6" />
-	  </inertial>
-	</link>
   </xacro:macro>
   <xacro:macro name="arlobot_standoff_5in" params="parent number x_loc y_loc z_loc">

File: Simulation/urdf/common_default.urdf.xacro (robot description, xacro)
@@ -1,21 +1,19 @@
 <?xml version="1.0"?>
 <robot name="arlobot" xmlns:xacro="http://ros.org/wiki/xacro">
-  <!-- A common file to tie together all of the bits and bobs of the entire robot
-  Modeled after turtlebot_description
-  NOTE: All Gazebo references are gone, so simulation will have to be rebuilt if you want it -->
-  <!-- From $(find turtlebot_description)/urdf/common_properties.urdf.xacro -->
-  <!-- It is required by asus_xtion_pro.urdf.xacro -->
   <xacro:property name="M_PI" value="3.1415926535897931"/>
-  <xacro:property name="camera_link" value="0.05" />
-  <!-- This is where the 3D camera location is set. -->
-  <xacro:include filename="$(find Simulation)/urdf/3d_camera_position.urdf.xacro"/>
+  <!-- Loading config for arlo and all sensors -->
+  <xacro:include filename="$(find Simulation)/urdf/camera.urdf.xacro"/>
+  <xacro:include filename="$(find Simulation)/urdf/lidar.urdf.xacro"/>
+  <xacro:include filename="$(find Simulation)/urdf/imu.urdf.xacro"/>
+  <xacro:include filename="$(find Simulation)/urdf/arlo_stack.urdf.xacro"/>
   <!-- ArloBot -->
-  <xacro:include filename="$(find Simulation)/urdf/arlo_2stack.urdf.xacro"/>
-  <!-- 3D Sensor -->
-  <!-- xacro:include filename="$(find Simulation)/urdf/asus_xtion_pro.urdf.xacro"-->
-	<!-- Lidar Plugin -->
-  <xacro:include filename="$(find Simulation)/urdf/arlobot.gazebo" />
+  <xacro:arlobot/>
+  <!--sensor init define parent frame here-->
+  <xacro:lidar parent="base_link"/>
+  <xacro:camera parent="base_link"/>
+  <xacro:imu parent="base_link"/>
+  <!-- sensor/actor plugins init -->
+  <xacro:include filename="$(find Simulation)/urdf/arlobot.gazebo"/>
+  <!--adding one additional plate-->
   <xacro:stack_circles parent="base_link"/>
-  <!--xacro:sensor_asus_xtion_pro parent="base_link"-->
-  <xacro:arlobot/>
 </robot>

Commit message: URDF andustments for robot localization

File: Simulation/urdf/arlo_stack.urdf.xacro (robot description, xacro)
@@ -223,5 +223,5 @@
         <origin xyz="0 0 0" rpy="0 ${M_PI/2} ${M_PI/2}"/>
         <geometry>
-          <cylinder radius="0.0762" length="0.03175"/>
+          <cylinder radius="0.0762" length="0.001"/>
         </geometry>
         <surface>
@@ -235,6 +235,4 @@
       </collision>
     </link>
-    <!-- Fixed because we never rotate it anyway, it is just for show -->
-    <!-- NOTE This may prevent gazebo from working with this model -->
     <joint name="left_wheel_joint" type="continuous">
       <origin xyz="0 0.01905 0" rpy="0 0 0"/>
@@ -261,5 +259,5 @@
         <origin xyz="0 0 0" rpy="0 ${M_PI/2} ${M_PI/2}"/>
         <geometry>
-          <cylinder radius="0.0762" length="0.03175"/>
+          <cylinder radius="0.0762" length="0.001"/>
         </geometry>
         <surface>

File: Simulation/urdf/camera.urdf.xacro (robot description, xacro)
@@ -1,6 +1,6 @@
 <?xml version="1.0"?>
 <robot xmlns:xacro="http://ros.org/wiki/xacro">
-	<xacro:property name="camera_angle" value="${45 *180/M_PI}" /><!--angle measured from horizontal downwards-->
-	<xacro:property name="camera_hight" value="${0.45-0.10125}" /><!--since this is relative to the base_link we have to substract 0.10125 from the hight we want-->
+	<xacro:property name="camera_angle" value="${70 *M_PI/180}" /><!--angle measured from horizontal downwards-->
+	<xacro:property name="camera_hight" value="${0.6-0.10125}" /><!--since this is relative to the base_link we have to substract 0.10125 from the hight we want-->
 	<xacro:property name="camera_xoffset" value="0.18" />
 	<xacro:macro name="camera" params="parent">
@@ -26,5 +26,5 @@
 		</link>
 		<joint name="camera_joint" type="fixed">
-			<axis xyz="0 1 0" />
+			<axis xyz="0 1 0"/>
 		    <origin xyz="${camera_xoffset} 0 ${camera_hight}" rpy="0 ${camera_angle} 0"/>
 		    <parent link="${parent}"/>

Commit message: Sync

File: Simulation/urdf/arlo_stack.urdf.xacro (robot description, xacro)
@@ -223,5 +223,5 @@
         <origin xyz="0 0 0" rpy="0 ${M_PI/2} ${M_PI/2}"/>
         <geometry>
-          <cylinder radius="0.0762" length="0.001"/>
+          <cylinder radius="0.0762" length="0.03175"/>
         </geometry>
         <surface>
@@ -259,5 +259,5 @@
         <origin xyz="0 0 0" rpy="0 ${M_PI/2} ${M_PI/2}"/>
         <geometry>
-          <cylinder radius="0.0762" length="0.001"/>
+          <cylinder radius="0.0762" length="0.03175"/>
         </geometry>
         <surface>
